File: Z80_Demo1.kicad_sch (KiCad schematic)
At the start: 21 parts, among them J1 Conn_01x02_Pin, SW1 SW_Push, SW2 SW_DIP_x04, U1 NE555P, U2 Z80CPU, U3 SST39SF010, U4 74LS32, U5 AS6C4008-55PCN, U6 74LS04, U7 74LS32

Commit message: Add README
Other:
- company: (none) -> Francisco Sedano
- title: (none) -> Z80 CPU board
Changed lines of the file:
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@@
 (kicad_sch (version 20230121) (generator eeschema)
   (paper "A4")
+  (title_block
+    (title "Z80 CPU board")
+    (date "2023-11-27")
+    (rev "0.1")
+    (company "Francisco Sedano")
+  )
   (junction (at 39.37 81.28) (diameter 0) (color 0 0 0 0)
   )
